File: hardware/Neewer/Neewer.kicad_sch (KiCad schematic)
At the start: 31 parts, among them J1 Screw_Terminal_01x03, J2 Screw_Terminal_01x03, J3 PSU, Q1 IRLZ44N, Q2 IRLZ44N, Q3 IRLZ44N, Q4 IRLZ44N

Commit message: Update kicad
Parts:
- removed D1, D2, D3, D4: BAT46, Diode_THT:D_DO-35_SOD27_P2.54mm_Vertical_KathodeUp, symbol Diode:BAT46
- added D1, D2, D3, D4: 1N5819, Diode_THT:D_DO-41_SOD81_P5.08mm_Vertical_AnodeUp, symbol Diode:1N5819
- R5: footprint Resistor_THT:R_Axial_DIN0207_L6.3mm_D2.5mm_P2.54mm_Vertical -> Resistor_THT:R_Axial_DIN0207_L6.3mm_D2.5mm_P15.24mm_Horizontal
Connections:
- net PWM1: now also D1.2 (A)
- net PWM2: now also D2.2 (A)
- net PWM3: now also D3.2 (A)
- net PWM4: now also D4.2 (A)
- net VCC: now also D1.1 (K), D2.1 (K), D3.1 (K), D4.1 (K)
